File: serpente_plug.kicad_pcb (KiCad board)
At the start: 2 copper layers, 28.8 x 22 mm, 27 parts, among them J1 USB_A, J2 Conn_Power, J3 Conn_GPIO, SW1 SW_RESET, U1 GD25Q32CNIGR, U2 MCP1700-3302E_SOT23, U3 ATSAMD21E18A

Commit message: Fix GPIO numbers, add BOM, update README
Connections:
- J3 pad 1: /GPIO0 -> /GPIO5
- J3 pad 2: /GPIO1 -> /GPIO4
- J3 pad 3: /GPIO2 -> /GPIO3
- J3 pad 4: /GPIO3 -> /GPIO2
- J3 pad 5: /GPIO4 -> /GPIO1
- J3 pad 6: /GPIO5 -> /GPIO0
- U3 pad 11: /GPIO1 -> /GPIO4
- U3 pad 12: /GPIO0 -> /GPIO5
- U3 pad 5: /GPIO5 -> /GPIO0
- U3 pad 6: /GPIO4 -> /GPIO1
- U3 pad 7: /GPIO3 -> /GPIO2
- U3 pad 8: /GPIO2 -> /GPIO3
Routing:
- net /GPIO5: track 8.95 -> 10.0 mm
- net /GPIO0: track 10.0 -> 8.95 mm
- net /GPIO4: track 7.04 -> 7.97 mm
- net /GPIO1: track 7.97 -> 7.04 mm
Other:
- board text added: "JLCJLCJLCJLC"
Changed lines of the file:
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@@
-(kicad_pcb (version 20171130) (host pcbnew 5.1.2)
+(kicad_pcb (version 20171130) (host pcbnew "(5.1.2)-2")
   (general
     (thickness 1.6)
-    (drawings 32)
+    (drawings 33)
     (tracks 258)
     (zones 0)
@@
     (pcbplotparams
       (layerselection 0x010fc_ffffffff)
-      (usegerberextensions false)
+      (usegerberextensions true)
       (usegerberattributes false)
       (usegerberadvancedattributes false)
@@
       (outputformat 1)
       (mirror false)
-      (drillshape 1)
+      (drillshape 0)
       (scaleselection 1)
-      (outputdirectory ""))
+      (outputdirectory "gerb_plug"))
   )
   (net 0 "")
@@
       (net 32 "Net-(U3-Pad13)"))
     (pad 12 smd roundrect (at -0.25 2.45 90) (size 0.25 0.8) (layers F.Cu F.Paste F.Mask) (roundrect_rratio 0.25)
-      (net 17 /GPIO0))
+      (net 12 /GPIO5))
     (pad 11 smd roundrect (at -0.75 2.45 90) (size 0.25 0.8) (layers F.Cu F.Paste F.Mask) (roundrect_rratio 0.25)
-      (net 16 /GPIO1))
+      (net 13 /GPIO4))
     (pad 10 smd roundrect (at -1.25 2.45 90) (size 0.25 0.8) (layers F.Cu F.Paste F.Mask) (roundrect_rratio 0.25)
       (net 2 GND))
@@
       (net 3 +3V3))
     (pad 8 smd roundrect (at -2.45 1.75 90) (size 0.8 0.25) (layers F.Cu F.Paste F.Mask) (roundrect_rratio 0.25)
+      (net 14 /GPIO3))
+    (pad 7 smd roundrect (at -2.45 1.25 90) (size 0.8 0.25) (layers F.Cu F.Paste F.Mask) (roundrect_rratio 0.25)
       (net 15 /GPIO2))
-    (pad 7 smd roundrect (at -2.45 1.25 90) (size 0.8 0.25) (layers F.Cu F.Paste F.Mask) (roundrect_rratio 0.25)
-      (net 14 /GPIO3))
     (pad 6 smd roundrect (at -2.45 0.75 90) (size 0.8 0.25) (layers F.Cu F.Paste F.Mask) (roundrect_rratio 0.25)
-      (net 13 /GPIO4))
+      (net 16 /GPIO1))
     (pad 5 smd roundrect (at -2.45 0.25 90) (size 0.8 0.25) (layers F.Cu F.Paste F.Mask) (roundrect_rratio 0.25)
-      (net 12 /GPIO5))
+      (net 17 /GPIO0))
     (pad 4 smd roundrect (at -2.45 -0.25 90) (size 0.8 0.25) (layers F.Cu F.Paste F.Mask) (roundrect_rratio 0.25)
       (net 33 "Net-(U3-Pad4)"))
@@
     (fp_line (start -0.635 -1.27) (end 1.27 -1.27) (layer F.Fab) (width 0.1))
     (pad 6 thru_hole oval (at 0 12.7) (size 1.7 1.7) (drill 1) (layers *.Cu *.Mask)
+      (net 17 /GPIO0))
+    (pad 5 thru_hole oval (at 0 10.16) (size 1.7 1.7) (drill 1) (layers *.Cu *.Mask)
+      (net 16 /GPIO1))
+    (pad 4 thru_hole oval (at 0 7.62) (size 1.7 1.7) (drill 1) (layers *.Cu *.Mask)
+      (net 15 /GPIO2))
+    (pad 3 thru_hole oval (at 0 5.08) (size 1.7 1.7) (drill 1) (layers *.Cu *.Mask)
+      (net 14 /GPIO3))
+    (pad 2 thru_hole oval (at 0 2.54) (size 1.7 1.7) (drill 1) (layers *.Cu *.Mask)
+      (net 13 /GPIO4))
+    (pad 1 thru_hole rect (at 0 0) (size 1.7 1.7) (drill 1) (layers *.Cu *.Mask)
       (net 12 /GPIO5))
-    (pad 5 thru_hole oval (at 0 10.16) (size 1.7 1.7) (drill 1) (layers *.Cu *.Mask)
-      (net 13 /GPIO4))
-    (pad 4 thru_hole oval (at 0 7.62) (size 1.7 1.7) (drill 1) (layers *.Cu *.Mask)
-      (net 14 /GPIO3))
-    (pad 3 thru_hole oval (at 0 5.08) (size 1.7 1.7) (drill 1) (layers *.Cu *.Mask)
-      (net 15 /GPIO2))
-    (pad 2 thru_hole oval (at 0 2.54) (size 1.7 1.7) (drill 1) (layers *.Cu *.Mask)
-      (net 16 /GPIO1))
-    (pad 1 thru_hole rect (at 0 0) (size 1.7 1.7) (drill 1) (layers *.Cu *.Mask)
-      (net 17 /GPIO0))
     (model ${KISYS3DMOD}/Connector_PinHeader_2.54mm.3dshapes/PinHeader_1x06_P2.54mm_Vertical.wrl
       (at (xyz 0 0 0))
@@
     (pad 2 connect rect (at 1.3 -5.15 270) (size 2 7.5) (layers F.Cu F.Mask)
       (net 10 /USB_D-))
+  )
+  (gr_text JLCJLCJLCJLC (at 113.7 56 90) (layer B.SilkS)
+    (effects (font (size 0.8 0.8) (thickness 0.15)) (justify mirror))
   )
   (gr_line (start 124.2 62) (end 124.2 66) (layer Edge.Cuts) (width 0.05))
@@
   (segment (start 134 65.5) (end 134 64.4) (width 0.25) (layer F.Cu) (net 11))
   (segment (start 134 64.4) (end 130.6 61) (width 0.25) (layer F.Cu) (net 11))
-  (segment (start 137.6 59.2) (end 136.4 58) (width 0.127) (layer F.Cu) (net 12))
-  (segment (start 136.4 58) (end 134.2 58) (width 0.127) (layer F.Cu) (net 12))
-  (segment (start 132.75 56.016284) (end 132.75 55.45) (width 0.127) (layer F.Cu) (net 12))
-  (segment (start 134.2 58) (end 133.716858 57.516858) (width 0.127) (layer F.Cu) (net 12))
-  (segment (start 139.5 59.2) (end 137.6 59.2) (width 0.127) (layer F.Cu) (net 12))
-  (segment (start 133.716858 57.516858) (end 133.716858 56.983142) (width 0.127) (layer F.Cu) (net 12))
-  (segment (start 133.716858 56.983142) (end 132.75 56.016284) (width 0.127) (layer F.Cu) (net 12))
-  (segment (start 138.16 56.66) (end 139.5 56.66) (width 0.127) (layer F.Cu) (net 13))
-  (segment (start 137.85401 56.35401) (end 138.16 56.66) (width 0.127) (layer F.Cu) (net 13))
-  (segment (start 133.65401 56.35401) (end 137.85401 56.35401) (width 0.127) (layer F.Cu) (net 13))
-  (segment (start 133.25 55.45) (end 133.25 55.95) (width 0.127) (layer F.Cu) (net 13))
-  (segment (start 133.25 55.95) (end 133.65401 56.35401) (width 0.127) (layer F.Cu) (net 13))
-  (segment (start 138.33 54.12) (end 139.5 54.12) (width 0.127) (layer F.Cu) (net 14))
-  (segment (start 136.35 56.1) (end 138.33 54.12) (width 0.127) (layer F.Cu) (net 14))
-  (segment (start 133.9 56.1) (end 136.35 56.1) (width 0.127) (layer F.Cu) (net 14))
-  (segment (start 133.75 55.45) (end 133.75 55.95) (width 0.127) (layer F.Cu) (net 14))
-  (segment (start 133.75 55.95) (end 133.9 56.1) (width 0.127) (layer F.Cu) (net 14))
-  (segment (start 139.42 51.58) (end 139.5 51.58) (width 0.127) (layer F.Cu) (net 15))
-  (segment (start 138.4 52.6) (end 139.42 51.58) (width 0.127) (layer F.Cu) (net 15))
-  (segment (start 138.4 53.3) (end 138.4 52.6) (width 0.127) (layer F.Cu) (net 15))
-  (segment (start 134.25 55.45) (end 136.25 55.45) (width 0.127) (layer F.Cu) (net 15))
-  (segment (start 136.25 55.45) (end 138.4 53.3) (width 0.127) (layer F.Cu) (net 15))
-  (segment (start 138.16 49.04) (end 139.5 49.04) (width 0.127) (layer F.Cu) (net 16))
-  (segment (start 136.8 50.4) (end 138.16 49.04) (width 0.127) (layer F.Cu) (net 16))
-  (segment (start 136.8 52.9) (end 136.8 50.4) (width 0.127) (layer F.Cu) (net 16))
-  (segment (start 134.95 53.75) (end 135.95 53.75) (width 0.127) (layer F.Cu) (net 16))
-  (segment (start 135.95 53.75) (end 136.8 52.9) (width 0.127) (layer F.Cu) (net 16))
-  (segment (start 138.15 46.5) (end 139.5 46.5) (width 0.127) (layer F.Cu) (net 17))
-  (segment (start 136.5 48.15) (end 138.15 46.5) (width 0.127) (layer F.Cu) (net 17))
-  (segment (start 136.5 52.7) (end 136.5 48.15) (width 0.127) (layer F.Cu) (net 17))
-  (segment (start 134.95 53.25) (end 135.95 53.25) (width 0.127) (layer F.Cu) (net 17))
-  (segment (start 135.95 53.25) (end 136.5 52.7) (width 0.127) (layer F.Cu) (net 17))
+  (segment (start 137.6 59.2) (end 136.4 58) (width 0.127) (layer F.Cu) (net 17))
+  (segment (start 136.4 58) (end 134.2 58) (width 0.127) (layer F.Cu) (net 17))
+  (segment (start 132.75 56.016284) (end 132.75 55.45) (width 0.127) (layer F.Cu) (net 17))
+  (segment (start 134.2 58) (end 133.716858 57.516858) (width 0.127) (layer F.Cu) (net 17))
+  (segment (start 139.5 59.2) (end 137.6 59.2) (width 0.127) (layer F.Cu) (net 17))
+  (segment (start 133.716858 57.516858) (end 133.716858 56.983142) (width 0.127) (layer F.Cu) (net 17))
+  (segment (start 133.716858 56.983142) (end 132.75 56.016284) (width 0.127) (layer F.Cu) (net 17))
+  (segment (start 138.16 56.66) (end 139.5 56.66) (width 0.127) (layer F.Cu) (net 16))
+  (segment (start 137.85401 56.35401) (end 138.16 56.66) (width 0.127) (layer F.Cu) (net 16))
+  (segment (start 133.65401 56.35401) (end 137.85401 56.35401) (width 0.127) (layer F.Cu) (net 16))
+  (segment (start 133.25 55.45) (end 133.25 55.95) (width 0.127) (layer F.Cu) (net 16))
+  (segment (start 133.25 55.95) (end 133.65401 56.35401) (width 0.127) (layer F.Cu) (net 16))
+  (segment (start 138.33 54.12) (end 139.5 54.12) (width 0.127) (layer F.Cu) (net 15))
+  (segment (start 136.35 56.1) (end 138.33 54.12) (width 0.127) (layer F.Cu) (net 15))
+  (segment (start 133.9 56.1) (end 136.35 56.1) (width 0.127) (layer F.Cu) (net 15))
+  (segment (start 133.75 55.45) (end 133.75 55.95) (width 0.127) (layer F.Cu) (net 15))
+  (segment (start 133.75 55.95) (end 133.9 56.1) (width 0.127) (layer F.Cu) (net 15))
+  (segment (start 139.42 51.58) (end 139.5 51.58) (width 0.127) (layer F.Cu) (net 14))
+  (segment (start 138.4 52.6) (end 139.42 51.58) (width 0.127) (layer F.Cu) (net 14))
+  (segment (start 138.4 53.3) (end 138.4 52.6) (width 0.127) (layer F.Cu) (net 14))
+  (segment (start 134.25 55.45) (end 136.25 55.45) (width 0.127) (layer F.Cu) (net 14))
+  (segment (start 136.25 55.45) (end 138.4 53.3) (width 0.127) (layer F.Cu) (net 14))
+  (segment (start 138.16 49.04) (end 139.5 49.04) (width 0.127) (layer F.Cu) (net 13))
+  (segment (start 136.8 50.4) (end 138.16 49.04) (width 0.127) (layer F.Cu) (net 13))
+  (segment (start 136.8 52.9) (end 136.8 50.4) (width 0.127) (layer F.Cu) (net 13))
+  (segment (start 134.95 53.75) (end 135.95 53.75) (width 0.127) (layer F.Cu) (net 13))
+  (segment (start 135.95 53.75) (end 136.8 52.9) (width 0.127) (layer F.Cu) (net 13))
+  (segment (start 138.15 46.5) (end 139.5 46.5) (width 0.127) (layer F.Cu) (net 12))
+  (segment (start 136.5 48.15) (end 138.15 46.5) (width 0.127) (layer F.Cu) (net 12))
+  (segment (start 136.5 52.7) (end 136.5 48.15) (width 0.127) (layer F.Cu) (net 12))
+  (segment (start 134.95 53.25) (end 135.95 53.25) (width 0.127) (layer F.Cu) (net 12))
+  (segment (start 135.95 53.25) (end 136.5 52.7) (width 0.127) (layer F.Cu) (net 12))
   (via (at 130.1 47.645994) (size 0.6) (drill 0.3) (layers F.Cu B.Cu) (net 18))
   (segment (start 130.105218 47.645994) (end 130.1 47.645994) (width 0.127) (layer F.Cu) (net 18))

Commit message: Final rev 2 release!
Parts:
- removed R7, R8: 22R, Resistor_SMD:R_0603_1608Metric
- added TP7: TP_RESET, TestPoint:TestPoint_Pad_D1.0mm, B.Cu at (125.9, 60.7)
- D3: value LED_ARGB -> LED_RBAG
- J2: footprint Connector_PinHeader_2.54mm:PinHeader_1x04_P2.54mm_Vertical -> Connector_PinHeader_2.54mm_Extra:PinHeader_1x04_P2.54mm_Vertical_Castellated
- J3: footprint Connector_PinHeader_2.54mm:PinHeader_1x06_P2.54mm_Vertical -> Connector_PinHeader_2.54mm_Extra:PinHeader_1x06_P2.54mm_Vertical_Castellated
- SW1: footprint Button_Switch_SMD:SW_SPST_B3U-1000P -> Button_Switch_SMD:SW_SPST_B3U-1000P-B
- moved TP5 4.40 mm to (123.4, 57.5)
- moved TP6 4.40 mm to (123.4, 54.5)
- moved C2 3.30 mm to (127.5, 51.0)
- moved C1 3.24 mm to (131.8, 60.7), turned to 0 degrees
- moved R3 2.50 mm to (140.5, 62.4)
- moved R6 1.80 mm to (127.5, 54.0)
- moved D1 1.32 mm to (128.0, 58.6), turned to 0 degrees
- moved J2 1.23 mm to (134.1, 64.3)
- moved D2 1.20 mm to (128.0, 60.5), turned to 0 degrees
- moved R1 1.00 mm to (137.5, 62.4)
- moved D3 1.00 mm to (139.0, 65.4)
- moved C3 0.63 mm to (134.4, 58.2), turned to 90 degrees
- moved U2 0.63 mm to (131.9, 58.2)
- moved TP3 0.56 mm to (139.8, 63.0)
- moved TP1 0.55 mm to (139.8, 65.5)
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Connections:
- net Net-(SW1-Pad2) renamed /~RESET~
- D3 pad 3: Net-(D3-Pad3) -> +3V3
- D3 pad 4: +3V3 -> Net-(D3-Pad4)
- J2 pad 3: +3V3 -> GND
- J2 pad 4: GND -> +3V3
- R2 pad 1: Net-(D3-Pad3) -> Net-(D3-Pad4)
- U3 pad 20: /LED_R -> /LED_G
- U3 pad 21: /LED_B -> /LED_R
- U3 pad 22: /LED_G -> /LED_B
- U3 pad 23: Net-(R7-Pad1) -> /USB_D-
- U3 pad 24: Net-(R8-Pad1) -> /USB_D+
Routing:
- net /~RESET~: track 8.53 -> 21.1 mm, vias 0 -> 3
- net GND: track 7.60 -> 18.5 mm, vias 5 -> 11
- net +5V: track 6.30 -> 11.3 mm
- net /LED_G: track 23.5 -> 27.1 mm
- net Net-(R7-Pad1): track 3.59 -> 0.00 mm
- net Net-(D3-Pad3): track 3.44 -> 0.00 mm
- net /GPIO4: track 7.97 -> 10.8 mm
- net Net-(D3-Pad4): track 0.00 -> 2.87 mm
- net /GPIO3: track 7.26 -> 10.1 mm
- net Net-(R8-Pad1): track 2.75 -> 0.00 mm
- net /GPIO5: track 10.0 -> 12.3 mm
- net /GPIO2: track 7.13 -> 9.39 mm
- net /GPIO1: track 7.04 -> 9.30 mm
- net VBUS: track 21.1 -> 23.2 mm
- net /GPIO0: track 8.95 -> 10.9 mm
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Other:
- board size 28.8 x 22 mm -> 29.5 x 22 mm
- board text added: "CLK"
- board text added: "DAT"
- board text added: "IN"
- board text added: "Plug"
- board text added: "RST"
- board text added: "Serpente R2"
- board text added: "USB"
- board text added: "V"
- board text removed: "C"
- board text removed: "G"
- board text removed: "JLCJLCJLCJLC"
- board text removed: "Serpente Plug"
- board text removed: "VIN"
- board text removed: "VUSB"
